File: PCB/sense-nest.kicad_sch (KiCad schematic)
At the start: 2 parts, among them U1 MOUDLE-SEEEDUINO-XIAO-ESP32C3, U2 AM2302

Commit message: update gitignore
Parts:
- added Brd1: SSD1306, SSD1306 128x64:128x64OLED, symbol SSD1306 128x64:SSD1306
Connections:
- net +3V3: now also Brd1.2 (VCC)
- net GND: now also Brd1.1 (GND)
- net at U1.5 (PA8_A4_D4_SDA): now also Brd1.4 (SDA)
- net at U1.6 (PA9_A5_D5_SCL): now also Brd1.3 (SCL)
